Commit message: first working version of aruco, c++

File: ardrone_vislab/ardrone_vislab_description/urdf/quadrotor_sensors.urdf.xacro (robot description, xacro)
@@ -29,5 +29,5 @@
     <include filename="$(find ardrone_vislab_description)/urdf/sensors/generic_camera.urdf.xacro" />
     <xacro:generic_camera name="bottom" sim_name="ardrone" parent="base_link" update_rate="60" res_x="640" res_y="360" image_format="R8G8B8" hfov="${81*M_PI/180}">
-      <origin xyz="0.15 0.0 0.0" rpy="0 -${M_PI/2} 0"/>
+      <origin xyz="0.15 0.0 0.0" rpy="0 ${M_PI/2} 0"/>
     </xacro:generic_camera>
 </robot>
