Commit message: Added a collision/bumper plugin to the ardrone

File: ardrone_vislab/cvg_sim_gazebo_plugins/urdf/quadrotor_sensors.urdf.xacro (robot description, xacro)
@@ -64,4 +64,17 @@
       </plugin>
     </gazebo>
+    <gazebo reference="base_link">
+      <sensor name="quadrotor_contact_sensor_sim" type="contact">
+        <always_on>true</always_on>
+        <update_rate>100.0</update_rate>
+        <contact>
+          <collision>base_link_collision</collision>
+        </contact>
+        <plugin name="quadrotor_bumper_sim" filename="libgazebo_ros_bumper.so">
+          <bumperTopicName>ardrone/bumper</bumperTopicName>
+          <frameName>base_link</frameName>
+        </plugin>
+      </sensor>
+    </gazebo>
   </xacro:macro>
 </robot>
